File: usb_to_can.brd (EAGLE design)
At the start: 37 x 48 mm, 37 parts, among them IC1 FT230XS, X1 MINI-USB_SHIELD5P4-32005-501

Commit message: updated part values and BOM
Parts:
- C1, C11, C24, C8: value .1uF -> .1 uF
- C10: value 1uF -> 1 uF
- C27, C29, C31, C32: value 100nF -> .1 uF
- C30: value 10uF -> 10 uF
- C41: value 15 nF -> .1 u
- C9: value 4.7 -> 4.7 uF
- R22: value 70 -> 200
Changed lines of the file:
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@@
 <attribute name="NAME" x="2.451" y="27.072" size="0.4064" layer="25" font="vector"/>
 </element>
-<element name="C9" library="rcl" package="C0402K" value="4.7" x="15.41" y="23.17" smashed="yes" rot="R180">
+<element name="C9" library="rcl" package="C0402K" value="4.7 uF" x="15.41" y="23.17" smashed="yes" rot="R180">
 <attribute name="NAME" x="15.75" y="22.425" size="0.5" layer="25" font="vector" rot="R180"/>
 </element>
-<element name="C10" library="rcl" package="C0402K" value="1uF" x="5.04" y="36.64" smashed="yes" rot="R90">
+<element name="C10" library="rcl" package="C0402K" value="1 uF" x="5.04" y="36.64" smashed="yes" rot="R90">
 <attribute name="NAME" x="3.815" y="36.14" size="0.5" layer="25" font="vector" rot="R90"/>
 </element>
-<element name="C27" library="rcl" package="C0402K" value="100nF" x="6.04" y="36.64" smashed="yes" rot="R90">
+<element name="C27" library="rcl" package="C0402K" value=".1 uF" x="6.04" y="36.64" smashed="yes" rot="R90">
 <attribute name="NAME" x="7.215" y="36.14" size="0.5" layer="25" font="vector" rot="R90"/>
 </element>
-<element name="C31" library="rcl" package="C0402K" value="100nF" x="19.34" y="34.73" smashed="yes" rot="R270">
+<element name="C31" library="rcl" package="C0402K" value=".1 uF" x="19.34" y="34.73" smashed="yes" rot="R270">
 <attribute name="NAME" x="19.125" y="33.47" size="0.5" layer="25" font="vector" rot="R270"/>
 </element>
-<element name="C32" library="rcl" package="C0402K" value="100nF" x="4.98" y="25.34" smashed="yes" rot="R180">
+<element name="C32" library="rcl" package="C0402K" value=".1 uF" x="4.98" y="25.34" smashed="yes" rot="R180">
 <attribute name="NAME" x="5.48" y="24.755" size="0.5" layer="25" font="vector" rot="R180"/>
 </element>
@@
 <attribute name="NAME" x="8.809" y="21.8015" size="0.4064" layer="25" rot="R180"/>
 </element>
-<element name="R22" library="rcl" package="R0402" value="70" x="11.58" y="22.5" smashed="yes">
+<element name="R22" library="rcl" package="R0402" value="200" x="11.58" y="22.5" smashed="yes">
 <attribute name="NAME" x="13.505" y="21.825" size="0.5" layer="25" font="vector" rot="R90"/>
 </element>
@@
 <attribute name="NAME" x="2.16" y="34.01" size="0.5" layer="25" font="vector" rot="R90"/>
 </element>
-<element name="C41" library="rcl" package="C0402K" value="15 nF" x="3.44" y="30.14" smashed="yes" rot="R180">
+<element name="C41" library="rcl" package="C0402K" value=".1 u" x="3.44" y="30.14" smashed="yes" rot="R180">
 <attribute name="NAME" x="3.94" y="31.155" size="0.5" layer="25" font="vector" rot="R180"/>
 </element>
@@
 <attribute name="OC_NEWARK" value="unknown" x="39.28" y="75.29" size="1.778" layer="27" rot="R90" display="off"/>
 </element>
-<element name="C8" library="rcl" package="C0402K" value=".1uF" x="29.04" y="22.71" smashed="yes" rot="R270">
+<element name="C8" library="rcl" package="C0402K" value=".1 uF" x="29.04" y="22.71" smashed="yes" rot="R270">
 <attribute name="NAME" x="29.625" y="23.05" size="0.5" layer="25" font="vector" rot="R270"/>
 </element>
-<element name="C11" library="rcl" package="C0402K" value=".1uF" x="29.53" y="32.46" smashed="yes" rot="R270">
+<element name="C11" library="rcl" package="C0402K" value=".1 uF" x="29.53" y="32.46" smashed="yes" rot="R270">
 <attribute name="NAME" x="29.315" y="35.2" size="0.5" layer="25" font="vector" rot="R270"/>
 </element>
@@
 <attribute name="NAME" x="25.75" y="16.8908" size="0.5" layer="25" font="vector"/>
 </element>
-<element name="C29" library="rcl" package="C0402K" value="100nF" x="19.08" y="12.47" smashed="yes" rot="R90">
+<element name="C29" library="rcl" package="C0402K" value=".1 uF" x="19.08" y="12.47" smashed="yes" rot="R90">
 <attribute name="NAME" x="18.495" y="11.17" size="0.5" layer="25" font="vector" rot="R90"/>
 <attribute name="VALUE" x="20.53" y="11.97" size="1.016" layer="27" rot="R90"/>
 </element>
-<element name="C30" library="rcl" package="C0402K" value="10uF" x="19.31" y="15.17" smashed="yes" rot="R90">
+<element name="C30" library="rcl" package="C0402K" value="10 uF" x="19.31" y="15.17" smashed="yes" rot="R90">
 <attribute name="NAME" x="18.725" y="14.03" size="0.5" layer="25" font="vector" rot="R90"/>
 <attribute name="VALUE" x="20.76" y="14.67" size="1.016" layer="27" rot="R90"/>
@@
 <attribute name="NAME" x="26.395" y="23.723" size="0.5" layer="25" font="vector" rot="R180"/>
 </element>
-<element name="C1" library="rcl" package="C0402K" value=".1uF" x="21.19" y="33.56" smashed="yes" rot="R270">
+<element name="C1" library="rcl" package="C0402K" value=".1 uF" x="21.19" y="33.56" smashed="yes" rot="R270">
 <attribute name="NAME" x="20.975" y="35.82" size="0.5" layer="25" font="vector" rot="R270"/>
 </element>
-<element name="C24" library="rcl" package="C0402K" value=".1uF" x="22.47" y="26.29" smashed="yes" rot="R90"/>
+<element name="C24" library="rcl" package="C0402K" value=".1 uF" x="22.47" y="26.29" smashed="yes" rot="R90"/>
 <element name="IC1" library="ftdichip" package="SSOP16" value="FT230XS" x="13.6" y="18.91" smashed="yes"/>
 <element name="CHOKE1" library="SparkFun-Passives" package="0603" value="600r" x="20.32" y="18.16" smashed="yes" rot="R270">
