File: usb_to_can.sch (EAGLE design)
At the start: 37 parts, among them IC1 FT230XS, X1 MINI-USB_SHIELD5P4-32005-501

Commit message: updated part values and BOM
Parts:
- C1, C11, C24, C8: value .1uF -> .1 uF
- C10: value 1uF -> 1 uF
- C27, C29, C31, C32: value 100nF -> .1 uF
- C30: value 10uF -> 10 uF
- C41: value 15 nF -> .1 u
- C9: value 4.7 -> 4.7 uF
- R22: value 70 -> 200
Changed lines of the file:
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@@
 <drawing>
 <settings>
-<setting alwaysvectorfont="yes"/>
+<setting alwaysvectorfont="no"/>
 <setting keepoldvectorfont="yes"/>
 <setting verticaltext="up"/>
@@
 <part name="U$3" library="BenLibrary" deviceset="STM32F446RET6" device=""/>
 <part name="CHOKE" library="SparkFun-Passives" deviceset="INDUCTOR" device="0603" value="600r"/>
-<part name="C9" library="rcl" deviceset="C-US" device="C0402K" value="4.7"/>
-<part name="C10" library="rcl" deviceset="C-US" device="C0402K" value="1uF"/>
-<part name="C27" library="rcl" deviceset="C-US" device="C0402K" value="100nF"/>
-<part name="C31" library="rcl" deviceset="C-US" device="C0402K" value="100nF"/>
-<part name="C32" library="rcl" deviceset="C-US" device="C0402K" value="100nF"/>
+<part name="C9" library="rcl" deviceset="C-US" device="C0402K" value="4.7 uF"/>
+<part name="C10" library="rcl" deviceset="C-US" device="C0402K" value="1 uF"/>
+<part name="C27" library="rcl" deviceset="C-US" device="C0402K" value=".1 uF"/>
+<part name="C31" library="rcl" deviceset="C-US" device="C0402K" value=".1 uF"/>
+<part name="C32" library="rcl" deviceset="C-US" device="C0402K" value=".1 uF"/>
 <part name="LED2" library="SparkFun-LED" deviceset="LED" device="0603" value="G"/>
-<part name="R22" library="rcl" deviceset="R-US_" device="R0402" value="70"/>
+<part name="R22" library="rcl" deviceset="R-US_" device="R0402" value="200"/>
 <part name="XT1" library="sc_usercreated" deviceset="CSTCE" device=""/>
-<part name="C41" library="rcl" deviceset="C-US" device="C0402K" value="15 nF"/>
+<part name="C41" library="rcl" deviceset="C-US" device="C0402K" value=".1 u"/>
 <part name="DC1" library="dc-dc-converter" deviceset="VA-*?" device="S" technology="1224"/>
-<part name="C8" library="rcl" deviceset="C-US" device="C0402K" value=".1uF"/>
-<part name="C11" library="rcl" deviceset="C-US" device="C0402K" value=".1uF"/>
+<part name="C8" library="rcl" deviceset="C-US" device="C0402K" value=".1 uF"/>
+<part name="C11" library="rcl" deviceset="C-US" device="C0402K" value=".1 uF"/>
 <part name="R3" library="rcl" deviceset="R-US_" device="R0402" value="120"/>
 <part name="VR1" library="sc_usercreated" deviceset="LM1117" device=""/>
 <part name="GND14" library="SparkFun-Aesthetics" deviceset="GND" device=""/>
-<part name="C29" library="rcl" deviceset="C-US" device="C0402K" value="100nF"/>
-<part name="C30" library="rcl" deviceset="C-US" device="C0402K" value="10uF"/>
+<part name="C29" library="rcl" deviceset="C-US" device="C0402K" value=".1 uF"/>
+<part name="C30" library="rcl" deviceset="C-US" device="C0402K" value="10 uF"/>
 <part name="U$4" library="BenLibrary" deviceset="MCP2561" device=""/>
 <part name="U$8" library="BenLibrary" deviceset="SI8410" device=""/>
-<part name="C1" library="rcl" deviceset="C-US" device="C0402K" value=".1uF"/>
-<part name="C24" library="rcl" deviceset="C-US" device="C0402K" value=".1uF"/>
+<part name="C1" library="rcl" deviceset="C-US" device="C0402K" value=".1 uF"/>
+<part name="C24" library="rcl" deviceset="C-US" device="C0402K" value=".1 uF"/>
 <part name="IC1" library="ftdichip" deviceset="FT230X" device="S"/>
 <part name="CHOKE1" library="SparkFun-Passives" deviceset="INDUCTOR" device="0603" value="600r"/>
